Commit message: Added meshes for collision and Visualization

File: moveit_simple/test/resources/kuka_kr210/kr210l150.urdf (robot description, URDF)
Before this commit: robot kuka_kr210, 12 links, 11 joints
Links:
- link base_link: geometry collision mesh filename=package://moveit_simple/test/resources/kuka_kr210/meshes/co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; visual mesh filename=package://moveit_simple/test/resources/kuka_kr210/meshes/vi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
- link link_1: geometry collision mesh filename=package://moveit_simple/test/resources/kuka_kr210/meshes/co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; visual mesh filename=package://moveit_simple/test/resources/kuka_kr210/meshes/vi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
- link link_2: geometry collision mesh filename=package://moveit_simple/test/resources/kuka_kr210/meshes/co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; visual mesh filename=package://moveit_simple/test/resources/kuka_kr210/meshes/vi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
- link link_3: geometry collision mesh filename=package://moveit_simple/test/resources/kuka_kr210/meshes/co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; visual mesh filename=package://moveit_simple/test/resources/kuka_kr210/meshes/vi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
- link link_4: geometry collision mesh filename=package://moveit_simple/test/resources/kuka_kr210/meshes/co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; visual mesh filename=package://moveit_simple/test/resources/kuka_kr210/meshes/vi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
- link link_5: geometry collision mesh filename=package://moveit_simple/test/resources/kuka_kr210/meshes/co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; visual mesh filename=package://moveit_simple/test/resources/kuka_kr210/meshes/vi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
- link link_6: geometry collision mesh filename=package://moveit_simple/test/resources/kuka_kr210/meshes/co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; visual mesh filename=package://moveit_simple/test/resources/kuka_kr210/meshes/vi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
