Commit message: Renamed and modified transformToolToEndLink(...) to transformPoseBetweenFrames(...) to address generic Pose conversions between frames and overrode getPose(...) to facilitate custom_tool_frames with the getPose(...) function -- Unit Tests successful

File: moveit_simple/test/resources/kuka_kr210/kuka_custom_tool.urdf (robot description, URDF)
Before this commit: robot kuka_custom_tool, 2 links, 1 joints
Joints:
- joint tool0-tool_custom: origin xyz=0.0 0.0 0.0 rpy=0 0 0 -> xyz=1.0 3.0 1.5 rpy=3.142 -0.964 3.142

Commit message: #Issue with addTrajPoint(...) that accepts a point without pose -- This commit is intended as a reference point for anyone attempting to resolve it, open rviz to visualize the problem

File: moveit_simple/test/resources/kuka_kr210/kuka_custom_tool.urdf (robot description, URDF)
Before this commit: robot kuka_custom_tool, 2 links, 1 joints
Joints:
- joint tool0-tool_custom: origin xyz=1.0 3.0 1.5 rpy=3.142 -0.964 3.142 -> xyz=0.0 0.0 0.5 rpy=0.0 0.0 0.0
