Commit message: Changed parent of wayouts to be world instead of base_link

File: moveit_simple/test/resources/motoman_mh5/urdf/motoman_mh5_robot_macro.xacro (robot description, xacro)
@@ -24,6 +24,6 @@
     <!-- Joints -->
     <joint name="${prefix}world_to_base" type="fixed">
-      <parent link="world"/>
-      <child link="${prefix}base_link"/>
+      <parent link="${prefix}base_link"/>
+      <child link="world"/>
       <origin rpy="0 0 0" xyz="0 0 0"/>
     </joint>
@@ -39,5 +39,5 @@
     </joint>
     <joint name="${prefix}tool_custom_joint" type="fixed">
-      <parent link="${prefix}tool0"/>
+      <parent link="${prefix}ee_link"/>
       <child link="${prefix}tool_custom"/>
       <origin rpy="0 0 0" xyz="0 0 0.15"/>
@@ -47,5 +47,5 @@
     <link name="wp1"/>
     <joint name="base-waypoint1" type="fixed">
-      <parent link="${prefix}base_link"/>
+      <parent link="world"/>
       <child link="wp1"/>
       <origin xyz="0.56 -0.023 0.821" rpy="0.000 -0.488 0.000"/>
@@ -53,5 +53,5 @@
     <link name="wp2"/>
     <joint name="base-waypoint2" type="fixed">
-      <parent link="${prefix}base_link"/>
+      <parent link="world"/>
       <child link="wp2"/>
       <origin xyz="-0.092 -0.094 0.852" rpy="3.142 0.0 3.142"/>
@@ -59,5 +59,5 @@
     <link name="wp3"/>
     <joint name="base-waypoint3" type="fixed">
-      <parent link="${prefix}base_link"/>
+      <parent link="world"/>
       <child link="wp3"/>
       <origin xyz="0.33 -0.306 0.825" rpy="0.000 0.000 0.228"/>
@@ -65,5 +65,5 @@
     <link name="wp4"/>
     <joint name="base-waypoint4" type="fixed">
-      <parent link="${prefix}base_link"/>
+      <parent link="world"/>
       <child link="wp4"/>
       <origin xyz="0.23 0.402 1.799" rpy="0.000 0.000 0.000"/>

Commit message: Adjusted waypoints

File: moveit_simple/test/resources/motoman_mh5/urdf/motoman_mh5_robot_macro.xacro (robot description, xacro)
@@ -49,5 +49,5 @@
       <parent link="world"/>
       <child link="wp1"/>
-      <origin xyz="0.56 -0.023 0.821" rpy="0.000 -0.488 0.000"/>
+      <origin xyz="0.3 -0.023 0.821" rpy="0.000 -0.488 0.000"/>
     </joint>
     <link name="wp2"/>
@@ -55,5 +55,5 @@
       <parent link="world"/>
       <child link="wp2"/>
-      <origin xyz="-0.092 -0.094 0.852" rpy="3.142 0.0 3.142"/>
+      <origin xyz="-0.35 -0.094 0.852" rpy="3.142 -1.5 3.142"/>
     </joint>
     <link name="wp3"/>

Commit message: Adjusted waypoints so they can be added to a trajectory without failing

File: moveit_simple/test/resources/motoman_mh5/urdf/motoman_mh5_robot_macro.xacro (robot description, xacro)
@@ -49,5 +49,5 @@
       <parent link="world"/>
       <child link="wp1"/>
-      <origin xyz="0.3 -0.023 0.821" rpy="0.000 -0.488 0.000"/>
+      <origin xyz="0.7 0.1 0.4" rpy="0.0 1.7 0.0"/>
     </joint>
     <link name="wp2"/>
@@ -55,5 +55,5 @@
       <parent link="world"/>
       <child link="wp2"/>
-      <origin xyz="-0.35 -0.094 0.852" rpy="3.142 -1.5 3.142"/>
+      <origin xyz="0.8 -0.1 0.2" rpy="0.0 2.3 0.0"/>
     </joint>
     <link name="wp3"/>
@@ -61,5 +61,5 @@
       <parent link="world"/>
       <child link="wp3"/>
-      <origin xyz="0.33 -0.306 0.825" rpy="0.000 0.000 0.228"/>
+      <origin xyz="0.65 0.0 0.9" rpy="0.0 1.2 0.0"/>
     </joint>
     <link name="wp4"/>

Commit message: Updated waypoints to be more reachable

File: moveit_simple/test/resources/motoman_mh5/urdf/motoman_mh5_robot_macro.xacro (robot description, xacro)
@@ -55,5 +55,5 @@
       <parent link="world"/>
       <child link="wp2"/>
-      <origin xyz="0.8 -0.1 0.2" rpy="0.0 2.3 0.0"/>
+      <origin xyz="0.65 -0.1 0.2" rpy="0.0 2.3 0.0"/>
     </joint>
     <link name="wp3"/>

Commit message: Added a translation between the world frame and base link of the robot

File: moveit_simple/test/resources/motoman_mh5/urdf/motoman_mh5_robot_macro.xacro (robot description, xacro)
@@ -26,5 +26,5 @@
       <parent link="${prefix}base_link"/>
       <child link="world"/>
-      <origin rpy="0 0 0" xyz="0 0 0"/>
+      <origin rpy="0 0 0" xyz="0.25 0 0"/>
     </joint>
     <joint name="${prefix}joint_t_tool0_joint" type="fixed">

Commit message: Made world the root frame instead of base link

File: moveit_simple/test/resources/motoman_mh5/urdf/motoman_mh5_robot_macro.xacro (robot description, xacro)
@@ -24,7 +24,7 @@
     <!-- Joints -->
     <joint name="${prefix}world_to_base" type="fixed">
-      <parent link="${prefix}base_link"/>
-      <child link="world"/>
-      <origin rpy="0 0 0" xyz="0.25 0 0"/>
+      <parent link="world"/>
+      <child link="${prefix}base_link"/>
+      <origin rpy="0 0 0" xyz="0.05 0 0"/>
     </joint>
     <joint name="${prefix}joint_t_tool0_joint" type="fixed">
